File: DC-DC_400W.kicad_pcb (KiCad board)
At the start: 2 copper layers, 77 x 63 mm, 12 parts, among them J1 Conn_01x24, J10 Conn_01x05, J2 Conn_01x03, J3 Conn_01x05, J5 Conn_01x01, J6 Conn_01x02, J7 Conn_01x01, J8 Conn_01x01, J9 Conn_01x01

Commit message: final test version
Parts:
- added J4: Conn_01x01, Mounting_Holes:MountingHole_3.2mm_M3_ISO7380_Pad, F.Cu at (118.3, 73.2)
- moved R1 3.87 mm to (123.2, 69.8)
- moved J5 2.50 mm to (94.8, 73.2)
- moved J7 2.50 mm to (163.8, 73.2)
- moved J8 2.50 mm to (94.8, 123.2)
- moved J9 2.50 mm to (163.8, 123.2)
Routing:
- net GND: track 224.1 -> 194.1 mm, vias 75 -> 39
- net /TRIM-: track 6.46 -> 9.82 mm
- net /TRIM+: track 5.95 -> 2.80 mm

Commit message: final 1.0 version
Parts:
- removed J10, J3: Conn_01x05, Connectors_Phoenix:PhoenixContact_MSTBVA-G_05x5.00mm_Vertical
- added G***: LOGO, custom:LOGO, F.Cu at (158.3, 85.0)
- added J11: Conn_01x06, Connectors_Phoenix:PhoenixContact_MSTBVA-G_06x5.00mm_Vertical, F.Cu at (135.1, 112.0)
- added J12: Conn_01x06, Connectors_Phoenix:PhoenixContact_MSTBVA-G_06x5.00mm_Vertical, F.Cu at (135.1, 124.1)
- added R3: 402R, Resistors_SMD:R_0603, F.Cu at (121.6, 69.8)
- R2: value 680R -> 560R
- moved J7 5.00 mm to (168.8, 73.1)
- moved J9 5.00 mm to (168.8, 123.4)
- moved J2 2.00 mm to (139.2, 88.0)
- moved D1 1.00 mm to (132.9, 79.2)
- moved J4 0.15 mm to (118.3, 73.1)
- moved J5 0.15 mm to (94.8, 73.1)
- moved J8 0.15 mm to (94.8, 123.4)
Routing:
- net GND: track 194.1 -> 201.6 mm
- net +12V: track 36.6 -> 34.6 mm
- net /TRIM-: track 9.82 -> 11.4 mm
- net /TRIM+: track 2.80 -> 4.42 mm
- net Net-(D1-Pad2): track 2.55 -> 1.55 mm
Other:
- board size 77 x 63 mm -> 82 x 63 mm
- board text added: "+12V"
- board text added: "DC/DC 400W v.1.0"
- board text added: "GND"
- board text added: "POWER_GOOD"

Commit message: 0.35mm/0.35mm
Routing:
- net GND: track 201.6 -> 190.7 mm
- net +12V: track 34.6 -> 35.3 mm
Other:
- net class Default: clearance 0.25 -> 0.35; trace_width 0.25 -> 0.35
- rule trace_clearance: 0.25 -> 0.35
- rule trace_min: 0.25 -> 0.35
